Commit message: 20240811

File: src/description/robot_description.urdf (robot description, URDF)
Before this commit: robot robot, 3 links, 2 joints
Links:
- added link lidar_link; visual cylinder length=0.055 radius=0.0508
Joints:
- added joint lidar_joint: type fixed, parent base_link, child lidar_link, origin xyz=0.05 0 0.03 rpy=0 0 0

Commit message: 20240811

File: src/description/robot_description.urdf (robot description, URDF)
Before this commit: robot robot, 4 links, 3 joints
Links:
- removed link lidar_link
- added link laser; visual cylinder length=0.055 radius=0.0508
Joints:
- joint lidar_joint: child lidar_link -> laser

Commit message: 20240813_1.1

File: src/description/robot_description.urdf (robot description, URDF)
Before this commit: robot robot, 4 links, 3 joints
Links:
- link front_caster: geometry visual sphere radius=${(wheel_radius+wheel_zoff)/2}

Commit message: 20240813_1.2

File: src/description/robot_description.urdf (robot description, URDF)
Before this commit: robot robot, 4 links, 3 joints
Joints:
- joint caster_joint: origin xyz=${caster_xoff} 0.0 ${-(base_height/2)} rpy=0 0 0 -> xyz=${caster_xoff} 0.0 ${-((wheel_radius+wheel_zoff)/2)} rpy=0 0 0

Commit message: 20240905

File: src/description/robot_description.urdf (robot description, URDF)
Before this commit: robot robot, 4 links, 3 joints
Links:
- added link imu_link; visual box size=0.045 0.06 0.01
Joints:
- added joint imu_joint: type fixed, parent base_link, child imu_link, origin xyz=${lidar_xoff} 0.0 ${base_height/2 + 0.005}

Commit message: 20250113

File: src/description/robot_description.urdf (robot description, URDF)
Before this commit: robot robot, 5 links, 4 joints
Links:
- link base_link: geometry collision box size=${base_length} ${base_width} ${base_height}; visual box size=${base_length} ${base_width} ${base_height}
- link front_caster: geometry collision sphere radius=${(wheel_radius+wheel_zoff-(base_height/2))}; visual sphere radius=${(wheel_radius+wheel_zoff-(base_height/2))}
- link imu_link: geometry collision box size=0.045 0.06 0.01; visual box size=0.045 0.06 0.01
- link laser: mass None -> 0.17; geometry collision cylinder length=0.06 radius=0.035; visual cylinder length=0.06 radius=0.035

Commit message: 20250125

File: src/description/robot_description.urdf (robot description, URDF)
Before this commit: robot robot, 5 links, 4 joints
Links:
- added link battery; collision box size=${battery_length} ${base_width} ${battery_height}; visual box size=${battery_length} ${base_width} ${battery_height}
- added link caster_base; collision box size=${caster_base_length} ${caster_base_width} ${caster_base_he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; visual box size=${caster_base_length} ${caster_base_width} ${caster_base_he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
- link front_caster: geometry collision sphere radius=${caster_radius}; visual sphere radius=${caster_radius}
Joints:
- added joint battery_joint: type fixed, parent base_link, child battery, origin xyz=${lidar_xoff} 0.0 ${base_height/2+battery_height/2}
- added joint caster_base_joint: type fixed, parent base_link, child caster_base, origin xyz=${caster_xoff} 0.0 -${base_height/2+caster_base_height/2}
- joint caster_joint: origin xyz=${caster_xoff} 0.0 ${-(base_height/2)} rpy=0 0 0 -> xyz=${caster_xoff} 0.0 -${caster_radius+caster_base_height+(base_height/2)} rpy=0 0 0
- joint imu_joint: origin xyz=${lidar_xoff} 0.0 ${base_height/2 + 0.005} -> xyz=${lidar_xoff} 0.0 ${base_height/2+battery_height+0.005}
- joint lidar_joint: origin xyz=${lidar_xoff} 0.0 ${base_height/2+lidar_height/2} rpy=0 0 0 -> xyz=${lidar_xoff} 0.0 ${base_height/2+battery_height+lidar_height/2} rpy=0 0 0

Commit message: 20250125

File: src/description/robot_description.urdf (robot description, URDF)
Before this commit: robot robot, 7 links, 6 joints
Links:
- added link raspi; collision box size=${raspi_length} ${raspi_width} ${raspi_height}; visual box size=${raspi_length} ${raspi_width} ${raspi_height}
- link battery: geometry collision box size=${battery_length} ${battery_width} ${battery_height}; visual box size=${battery_length} ${battery_width} ${battery_height}
Joints:
- added joint raspi_joint: type fixed, parent base_link, child raspi, origin xyz=-${raspi_xoff} 0.0 ${base_height/2+raspi_height/2}

Commit message: 20250126

File: src/description/robot_description.urdf (robot description, URDF)
Before this commit: robot robot, 8 links, 7 joints
Links:
- link imu_link: geometry collision box size=${imu_length} ${imu_width} ${imu_height}; visual box size=${imu_length} ${imu_width} ${imu_height}
- link laser: mass 0.17 -> ${lidar_mass}; geometry collision cylinder length=${lidar_height} radius=${lidar_radius}; visual cylinder length=${lidar_height} radius=${lidar_radius}
Joints:
- joint imu_joint: origin xyz=${lidar_xoff} 0.0 ${base_height/2+battery_height+0.005} -> xyz=${lidar_xoff} 0.0 ${base_height/2+battery_height+imu_height/2}
