Commit message: 20250531

File: src/description/robot_description_ign.urdf (robot description, URDF)
Before this commit: robot robot, 8 links, 7 joints
Links:
- added link camera_link; collision box size=${camera_length} ${camera_width} ${camera_height}; visual box size=${camera_length} ${camera_width} ${camera_height}
Joints:
- added joint camera_joint: type fixed, parent base_link, child camera_link, origin xyz=${camera_xoff} 0.0 ${base_height/2+battery_height+camera_height/2}
